File: guitar-input-eg/guitar-input-eg.kicad_pcb (KiCad board)
At the start: 2 copper layers, 39.1 x 38.1 mm, 33 parts, among them U1 TL074, U2 TL072, U3 TL074, U4 TL074, U5 TL074, U6 TL072

Commit message: finished the mod synth :D
(i keep on forgetting to commit :sob:)
Parts:
- added .: LOGO, LOGO, B.Cu at (85.5, 42.6)
Connections:
- C1 pad 2: Net-(U3A--) -> Net-(U3B-+)
- C4 pad 1: Net-(U6A--) -> Net-(U6B--)
- GAIN1 pad 1: Net-(D3-K) -> Net-(GAIN1-Pad1)
- GAIN1 pad 3: Net-(GAIN1-Pad3) -> Net-(D3-K)
- GAIN2 pad 2: Net-(U5A--) -> Net-(U5D--)
- GAIN3 pad 2: Net-(U6A-+) -> Net-(U6B-+)
- GAIN4 pad 3: Net-(U4A-+) -> Net-(U4A--)
- R10 pad 2: Net-(U1A--) -> Net-(U1C--)
- R11 pad 1: Net-(GAIN1-Pad3) -> Net-(GAIN1-Pad1)
- R5 pad 2: Net-(U3A--) -> Net-(U3B-+)
- R7 pad 2: Net-(U4A-+) -> Net-(U4A--)
- R8 pad 2: Net-(U4A--) -> Net-(U4A-+)
- R9 pad 1: Net-(U4A--) -> Net-(U4A-+)
- U1 pad 1: Net-(U1A--) -> (no net)
- U1 pad 10: (no net) -> Net-(D3-K)
- U1 pad 2: Net-(U1A--) -> (no net)
- U1 pad 3: Net-(D3-K) -> (no net)
- U1 pad 8: (no net) -> Net-(U1C--)
- U1 pad 9: (no net) -> Net-(U1C--)
- U3 pad 1: Net-(D3-A) -> (no net)
- U3 pad 2: Net-(U3A--) -> (no net)
- U3 pad 3: Net-(D3-A) -> (no net)
- U3 pad 5: (no net) -> Net-(U3B-+)
- U3 pad 6: (no net) -> Net-(D3-A)
- U3 pad 7: (no net) -> Net-(D3-A)
- U5 pad 1: Net-(D5-A) -> (no net)
- U5 pad 12: (no net) -> Net-(U1C--)
- U5 pad 13: (no net) -> Net-(U5D--)
- U5 pad 14: (no net) -> Net-(D5-A)
- U5 pad 2: Net-(U5A--) -> (no net)
- U5 pad 3: Net-(U1A--) -> (no net)
- U6 pad 1: Net-(U6A--) -> (no net)
- U6 pad 2: Net-(U6A--) -> (no net)
- U6 pad 3: Net-(U6A-+) -> (no net)
- U6 pad 5: (no net) -> Net-(U6B-+)
- U6 pad 6: (no net) -> Net-(U6B--)
- U6 pad 7: (no net) -> Net-(U6B--)
Routing:
- net Net-(U6B-+): track 0.00 -> 39.3 mm, vias 0 -> 1
- net Net-(U6A-+): track 34.0 -> 0.00 mm, vias 1 -> 0
- net Net-(U4A--): track 38.8 -> 8.98 mm, vias 2 -> 0
- net Net-(U4A-+): track 8.55 -> 36.9 mm
- net Net-(U1A--): track 22.8 -> 0.00 mm, vias 2 -> 0
- net Net-(U6B--): track 0.00 -> 20.9 mm, vias 0 -> 2
- net Net-(U1C--): track 0.00 -> 20.6 mm
- net Net-(U3B-+): track 0.00 -> 19.2 mm, vias 0 -> 2
- net Net-(U5D--): track 0.00 -> 16.1 mm
- net GND: track 6.83 -> 22.6 mm, vias 1 -> 7
- net Net-(U6A--): track 15.4 -> 0.00 mm, vias 2 -> 0
- net Net-(U3A--): track 12.9 -> 0.00 mm
- net Net-(U5A--): track 10.7 -> 0.00 mm
- net Net-(GAIN1-Pad1): track 0.00 -> 8.78 mm, vias 0 -> 2
- net Net-(D5-A): track 38.9 -> 30.8 mm, vias 2 -> 3
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Other:
- board text added: "guitar input"
