File: guitar-input-eg/guitar-input-eg.kicad_sch (KiCad schematic)
At the start: 33 parts, among them U1 TL074, U2 TL072, U3 TL074, U4 TL074, U5 TL074, U6 TL072

Commit message: finished the mod synth :D
(i keep on forgetting to commit :sob:)
Connections:
- net at C3.2, D3.1 (K), GAIN1.2: now also GAIN1.3, U1.10 (+); no longer GAIN1.1, U1.3 (+)
- net at R11.1: now also GAIN1.1; no longer GAIN1.3
- net at R8.2, R9.1: now also U4.3 (+); no longer U4.2 (-)
- net at GAIN4.3, R7.2: now also U4.2 (-); no longer U4.3 (+)
- net at GAIN2.2: now also U5.13 (-); no longer U5.2 (-)
- net at D3.2 (A), R6.1, U2.3 (+): now also U3.6 (-), U3.7; no longer U3.1, U3.3 (+)
- net at C1.2, R5.2: now also U3.5 (+); no longer U3.2 (-)
- net at D5.2 (A), R12.1: now also U5.14; no longer U5.1
- net at GAIN3.2: now also U6.5 (+); no longer U6.3 (+)
- new net: R10.2, U1.8, U1.9 (-), U5.12 (+)
- new net: C4.1, U6.6 (-), U6.7
Other:
- moved on the sheet: GAIN3
