File: square-vco/squarevco.kicad_pcb (KiCad board)
At the start: 2 copper layers, 64.1 x 41 mm, 40 parts, among them J4 Conn_01x10_Pin, J5 AudioJack3_SwitchT, U1 PIC12F683-xMC, U2 TL074, U3 L7805, U4 TL074, U5 TL074, U6 TL074, Y1 20mhz

Commit message: finished the mod synth :D
(i keep on forgetting to commit :sob:)
Parts:
- added J1: AudioJack4, Connector_Audio:Jack_3.5mm_QingPu_WQP-PJ398SM_Vertical_CircularHoles, F.Cu at (122.6, 97.4)
- added J1: AudioJack2_Dual_Switch, Connector_Audio:Jack_3.5mm_QingPu_WQP-PJ398SM_Vertical_CircularHoles, F.Cu at (5.03, 1.45)
- R6: value 100K -> 1M
Connections:
- 25K1 pad 1: Net-(U5A--) -> Net-(U5B--)
- B100K1 pad 1: +5V -> GND
- B100K1 pad 3: GND -> +5V
- FINE1 pad 1: +5V -> GND
- FINE1 pad 3: GND -> +5V
- R1 pad 2: Net-(U4A-+) -> Net-(U4D-+)
- R16 pad 1: Net-(U5A--) -> Net-(U5B--)
- R17 pad 2: Net-(U5A--) -> Net-(U5B--)
- R18 pad 1: Net-(U5A--) -> Net-(U5B--)
- R2 pad 1: Net-(U4A-+) -> Net-(U4D-+)
- R3 pad 1: Net-(U4A--) -> Net-(U4D--)
- R3 pad 2: unconnected-(R3-Pad2) -> GND
- R6 pad 2: Net-(U5A--) -> Net-(U5B--)
- R7 pad 1: Net-(U2A--) -> Net-(U2C--)
- R8 pad 1: Net-(U2A--) -> Net-(U2C--)
- U2 pad 1: Net-(R1-Pad1) -> (no net)
- U2 pad 10: (no net) -> Net-(U1-GP1)
- U2 pad 2: Net-(U2A--) -> (no net)
- U2 pad 3: Net-(U1-GP1) -> (no net)
- U2 pad 8: (no net) -> Net-(R1-Pad1)
- U2 pad 9: (no net) -> Net-(U2C--)
- U4 pad 1: Net-(U4A--) -> (no net)
- U4 pad 12: (no net) -> Net-(U4D-+)
- U4 pad 13: (no net) -> Net-(U4D--)
- U4 pad 14: (no net) -> Net-(U4D--)
- U4 pad 2: Net-(U4A--) -> (no net)
- U4 pad 3: Net-(U4A-+) -> (no net)
- U5 pad 1: Net-(R14-Pad1) -> (no net)
- U5 pad 2: Net-(U5A--) -> (no net)
- U5 pad 3: GND -> (no net)
- U5 pad 5: (no net) -> GND
- U5 pad 6: (no net) -> Net-(U5B--)
- U5 pad 7: (no net) -> Net-(R14-Pad1)
Routing:
- net GND: track 180.3 -> 42.5 mm, vias 4 -> 7
- net Net-(U5B--): track 0.00 -> 85.6 mm, vias 0 -> 3
- net Net-(R14-Pad1): track 6.20 -> 82.6 mm, vias 0 -> 2
- net Net-(U5A--): track 76.4 -> 0.00 mm, vias 1 -> 0
- net Net-(J4-Pin_1): track 22.0 -> 86.5 mm, vias 0 -> 1
- net Net-(J4-Pin_10): track 38.0 -> 92.2 mm, vias 0 -> 1
- net Net-(U2C--): track 0.00 -> 22.5 mm, vias 0 -> 2
- net Net-(U2A--): track 19.7 -> 0.00 mm
- net (no net): track 0.00 -> 17.8 mm, vias 0 -> 3
- net Net-(U4D-+): track 0.00 -> 17.1 mm
- net Net-(R1-Pad1): track 4.56 -> 18.7 mm, vias 0 -> 2
- net Net-(U4A-+): track 12.1 -> 0.00 mm
- net Net-(U4D--): track 0.00 -> 9.95 mm
- net Net-(U1-GP1): track 6.21 -> 12.2 mm
- net Net-(U4A--): track 4.50 -> 0.00 mm
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- added copper zone on B.Cu, net GND
- added copper zone on F.Cu, net GND
Other:
- board size 64.1 x 41 mm -> 65.2 x 41.2 mm
- board text added: "V1PERMODSYNTH SQUARE VCO"
