File: square-vco/squarevco.kicad_sch (KiCad schematic)
At the start: 39 parts, among them J4 Conn_01x10_Pin, J5 AudioJack3_SwitchT, U1 PIC12F683-xMC, U2 TL074, U3 L7805, U4 TL074, U5 TL074, U6 TL074, Y1 20mhz

Commit message: finished the mod synth :D
(i keep on forgetting to commit :sob:)
Parts:
- removed J5: AudioJack3_SwitchT, Connector_Audio:Jack_3.5mm_QingPu_WQP-PJ398SM_Vertical_CircularHoles, symbol Connector_Audio:AudioJack3_SwitchT
- added J1: AudioJack4, Connector_Audio:Jack_3.5mm_QingPu_WQP-PJ398SM_Vertical_CircularHoles, symbol Connector_Audio:AudioJack4
- R6: value 100K -> 1M
Connections:
- net +5V: now also B100K1.3, FINE1.3; no longer B100K1.1, FINE1.1
- net GND: now also B100K1.1, FINE1.1, U5.5 (+), J1.R1, J1.R2; no longer B100K1.3, FINE1.3, U5.3 (+)
- net at R1.2, R2.1: now also U4.12 (+); no longer U4.3 (+)
- net at 25K1.1, R16.1, R17.2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: now also U5.6 (-); no longer U5.2 (-)
- net at J4.10 (Pin_10), J4.9 (Pin_9), R11.2: now also J1.T
- net at R14.1, R16.2: now also U5.7; no longer U5.1
- net at R1.1: now also U2.8; no longer U2.1
- net at U1.6 (GP1): now also U2.10 (+); no longer U2.3 (+)
- net at J4.1 (Pin_1), J4.2 (Pin_2), R10.1: now also J1.S
- net at R7.1, R8.1: now also U2.9 (-); no longer U2.2 (-)
- new net: R3.1, U4.13 (-), U4.14
- no-connect marks 4 -> 5
Changed lines of the file:
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@@
 	)
 	(junction
+		(at 86.36 43.18)
+		(diameter 0)
+		(color 0 0 0 0)
+	)
+	(junction
 		(at 195.58 101.6)
 		(diameter 0)
@@
 	)
 	(junction
+		(at 40.64 41.91)
+		(diameter 0)
+		(color 0 0 0 0)
+	)
+	(junction
 		(at 101.6 50.8)
 		(diameter 0)
@@
 	)
 	(junction
-		(at 86.36 45.72)
-		(diameter 0)
-		(color 0 0 0 0)
-	)
-	(junction
 		(at 158.75 120.65)
 		(diameter 0)
@@
 	)
 	(junction
-		(at 171.45 120.65)
+		(at 86.36 40.64)
 		(diameter 0)
 		(color 0 0 0 0)
 	)
 	(junction
-		(at 54.61 43.18)
+		(at 171.45 120.65)
 		(diameter 0)
 		(color 0 0 0 0)
 	)
 	(junction
-		(at 86.36 40.64)
+		(at 54.61 43.18)
 		(diameter 0)
 		(color 0 0 0 0)
@@
 	)
 	(no_connect
+		(at 40.64 43.18)
+	)
+	(no_connect
 		(at 104.14 152.4)
 	)
@@
 	(wire
 		(pts
-			(xy 83.82 45.72) (xy 86.36 45.72)
+			(xy 107.95 138.43) (xy 107.95 140.97)
 		)
 		(stroke
@@
 		)
 	)
-	(wire
+	(bus
 		(pts
-			(xy 107.95 138.43) (xy 107.95 140.97)
+			(xy 24.13 24.13) (xy 121.92 24.13)
 		)
 		(stroke
@@
 		)
 	)
-	(bus
+	(wire
 		(pts
-			(xy 24.13 24.13) (xy 121.92 24.13)
+			(xy 158.75 129.54) (xy 158.75 132.08)
 		)
 		(stroke
@@
 	(wire
 		(pts
-			(xy 158.75 129.54) (xy 158.75 132.08)
+			(xy 88.9 140.97) (xy 88.9 144.78)
 		)
 		(stroke
@@
 	(wire
 		(pts
-			(xy 88.9 140.97) (xy 88.9 144.78)
+			(xy 40.64 41.91) (xy 40.64 43.18)
 		)
 		(stroke
@@
 	(wire
 		(pts
+			(xy 86.36 40.64) (xy 86.36 43.18)
+		)
+		(stroke
+			(width 0)
+			(type default)
+		)
+	)
+	(wire
+		(pts
 			(xy 120.65 123.19) (xy 121.92 123.19)
 		)
@@
 		)
 	)
-	(wire
-		(pts
-			(xy 86.36 40.64) (xy 73.66 40.64)
-		)
-		(stroke
-			(width 0)
-			(type default)
-		)
-	)
 	(bus
 		(pts
@@
 	(wire
 		(pts
-			(xy 86.36 48.26) (xy 86.36 50.8)
+			(xy 86.36 45.72) (xy 86.36 50.8)
 		)
 		(stroke
@@
 	(wire
 		(pts
+			(xy 73.66 40.64) (xy 86.36 40.64)
+		)
+		(stroke
+			(width 0)
+			(type default)
+		)
+	)
+	(wire
+		(pts
 			(xy 88.9 140.97) (xy 91.44 140.97)
 		)
@@
 	(wire
 		(pts
-			(xy 176.53 96.52) (xy 176.53 105.41)
+			(xy 83.82 43.18) (xy 86.36 43.18)
 		)
 		(stroke
@@
 	(wire
 		(pts
-			(xy 86.36 40.64) (xy 86.36 45.72)
+			(xy 176.53 96.52) (xy 176.53 105.41)
 		)
 		(stroke
@@
 		(lib_id "Amplifier_Operational:TL074")
 		(at 99.06 123.19 0)
-		(unit 1)
+		(unit 2)
 		(exclude_from_sim no)
 		(in_bom yes)
@@
 				(path "/c79140f3-880f-46a0-9cef-8ec1f2cc78f0"
 					(reference "U5")
-					(unit 1)
+					(unit 2)
 				)
 			)
@@
 	)
 	(symbol
+		(lib_id "Connector_Audio:AudioJack4")
+		(at 91.44 43.18 180)
+		(unit 1)
+		(exclude_from_sim no)
+		(in_bom yes)
+		(on_board yes)
+		(dnp no)
+		(fields_autoplaced yes)
+		(property "Reference" "J1"
+			(at 100.33 40.0049 0)
+			(effects
+				(font
+					(size 1.27 1.27)
+				)
+				(justify right)
+			)
+		)
+		(property "Value" "AudioJack4"
+			(at 100.33 42.5449 0)
+			(effects
+				(font
+					(size 1.27 1.27)
+				)
+				(justify right)
+			)
+		)
+		(property "Footprint" "Connector_Audio:Jack_3.5mm_QingPu_WQP-PJ398SM_Vertical_CircularHoles"
+			(at 91.44 43.18 0)
+			(effects
+				(font
+					(size 1.27 1.27)
+				)
+				(hide yes)
+			)
+		)
+		(property "Datasheet" "~"
+			(at 91.44 43.18 0)
+			(effects
+				(font
+					(size 1.27 1.27)
+				)
+				(hide yes)
+			)
+		)
+		(property "Description" "Audio Jack, 4 Poles (TRRS)"
+			(at 91.44 43.18 0)
+			(effects
+				(font
+					(size 1.27 1.27)
+				)
+				(hide yes)
+			)
+		)
+		(pin "R1"
+		)
+		(pin "S"
+		)
+		(pin "T"
+		)
+		(pin "R2"
+		)
+		(instances
+			(project ""
+				(path "/c79140f3-880f-46a0-9cef-8ec1f2cc78f0"
+					(reference "J1")
+					(unit 1)
+				)
+			)
+		)
+	)
+	(symbol
 		(lib_id "Device:R")
 		(at 195.58 97.79 0)
@@
 		(lib_id "Device:R_Potentiometer")
 		(at 72.39 140.97 0)
+		(mirror x)
 		(unit 1)
 		(exclude_from_sim no)
@@
 				)
 				(justify right)
+				(hide yes)
 			)
 		)
@@
 		(lib_id "Amplifier_Operational:TL074")
 		(at 212.09 104.14 0)
-		(unit 1)
+		(unit 4)
 		(exclude_from_sim no)
 		(in_bom yes)
@@
 				(path "/c79140f3-880f-46a0-9cef-8ec1f2cc78f0"
 					(reference "U4")
-					(unit 1)
+					(unit 4)
 				)
 			)
@@
 			)
 		)
-		(property "Value" "100K"
+		(property "Value" "1M"
 			(at 82.55 138.43 90)
 			(effects
@@
 		(lib_id "Amplifier_Operational:TL074")
 		(at 184.15 93.98 0)
-		(unit 1)
+		(unit 3)
 		(exclude_from_sim no)
 		(in_bom yes)
@@
 				(path "/c79140f3-880f-46a0-9cef-8ec1f2cc78f0"
 					(reference "U2")
-					(unit 1)
+					(unit 3)
 				)
 			)
@@
 	)
 	(symbol
-		(lib_id "Connector_Audio:AudioJack3_SwitchT")
-		(at 91.44 45.72 180)
-		(unit 1)
-		(exclude_from_sim no)
-		(in_bom yes)
-		(on_board yes)
-		(dnp no)
-		(property "Reference" "J5"
-			(at 99.06 41.2749 0)
-			(effects
-				(font
-					(size 1.27 1.27)
-				)
-				(justify right)
-				(hide yes)
-			)
-		)
-		(property "Value" "AudioJack3_SwitchT"
-			(at 97.028 46.228 0)
-			(effects
-				(font
-					(size 1.27 1.27)
-				)
-				(justify right)
-				(hide yes)
-			)
-		)
-		(property "Footprint" "Connector_Audio:Jack_3.5mm_QingPu_WQP-PJ398SM_Vertical_CircularHoles"
-			(at 91.44 45.72 0)
-			(effects
-				(font
-					(size 1.27 1.27)
-				)
-				(hide yes)
-			)
-		)
-		(property "Datasheet" "~"
-			(at 91.44 45.72 0)
-			(effects
-				(font
-					(size 1.27 1.27)
-				)
-				(hide yes)
-			)
-		)
-		(property "Description" "Audio Jack, 3 Poles (Stereo / TRS), Switched T Pole (Normalling)"
-			(at 91.44 45.72 0)
-			(effects
-				(font
-					(size 1.27 1.27)
-				)
-				(hide yes)
-			)
-		)
-		(pin "R"
-		)
-		(pin "T"
-		)
-		(pin "TN"
-		)
-		(pin "S"
-		)
-		(instances
-			(project ""
-				(path "/c79140f3-880f-46a0-9cef-8ec1f2cc78f0"
-					(reference "J5")
-					(unit 1)
-				)
-			)
-		)
-	)
-	(symbol
 		(lib_id "power:+5V")
 		(at 30.48 33.02 0)
@@
 		(lib_id "Device:R_Potentiometer")
 		(at 73.66 125.73 0)
+		(mirror x)
 		(unit 1)
 		(exclude_from_sim no)
@@
 				)
 				(justify right)
+				(hide yes)
 			)
 		)
@@
 	(symbol
 		(lib_id "power:GND")
-		(at 83.82 45.72 0)
+		(at 83.82 43.18 0)
 		(unit 1)
 		(exclude_from_sim no)
@@
 		(dnp no)
 		(property "Reference" "#PWR011"
-			(at 83.82 52.07 0)
+			(at 83.82 49.53 0)
 			(effects
 				(font
@@
 		)
 		(property "Value" "GND"
-			(at 83.82 49.53 0)
+			(at 83.82 46.99 0)
 			(effects
 				(font
@@
 		)
 		(property "Footprint" ""
-			(at 83.82 45.72 0)
+			(at 83.82 43.18 0)
 			(effects
 				(font
@@
 		)
 		(property "Datasheet" ""
-			(at 83.82 45.72 0)
+			(at 83.82 43.18 0)
 			(effects
 				(font
@@
 		)
 		(property "Description" "Power symbol creates a global label with name \"GND\" , ground"
-			(at 83.82 45.72 0)
+			(at 83.82 43.18 0)
 			(effects
 				(font
