File: vca/Untitled.kicad_sch (KiCad schematic)
At the start: 116 parts, among them J1 AudioJack4, J10 V-, J11 V-, J12 V-, J13 V+, J14 V+, J15 V+, J2 Conn_01x10_Pin, J4 Conn_01x04_Pin, J6 V+, J7 V+, J8 V-, J9 V-, Q1 2N3906, Q2 2N3906, Q3 2N3906, Q4 2N3906, U1 LM13700, U10 LM13700, U11 TL072, U12 LM13700, U13 TL072, U2 TL074, U3 TL074, U4 LM7805_TO220, U5 TL072, U6 TL074, U7 TL074, U8 LM13700, U9 TL072

Commit message: finished the mod synth :D
(i keep on forgetting to commit :sob:)
Parts:
- removed J10, J11, J12, J9: V-, Connector_PinHeader_2.54mm:PinHeader_1x01_P2.54mm_Vertical, symbol Connector:Conn_01x01_Pin
- removed J13, J14, J6, J7: V+, Connector_PinHeader_2.54mm:PinHeader_1x01_P2.54mm_Vertical, symbol Connector:Conn_01x01_Pin
- added unit 5 of U2
- added unit 5 of U3
- added unit 3 of U5
- added unit 3 of U9
- renumbered U7 to U7C1
Connections:
- net +15V: now also U2.4 (V+), U3.4 (V+), U5.8 (V+), U9.8 (V+)
- net GND: now also AMP1.1, AMP2.1, AMP3.1, AMP4.1, U2.5 (+), U3.5 (+), U6.3 (+), U6.5 (+), U7C1.5 (+), U2.11 (V-), U3.11 (V-), U5.4 (V-), U9.4 (V-); no longer AMP1.3, AMP2.3, AMP3.3, AMP4.3, U2.3 (+), U3.3 (+), U6.3 (+), U7C1.3 (+)
- net at D2.1 (K), R39.1, R40.1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: now also U6.6 (-); no longer U6.2 (-)
- net at D2.2 (A), Q3.2 (B): now also U6.7; no longer U6.1
- net at D3.2 (A), Q4.2 (B): now also U7C1.7; no longer U7C1.1
- net at D3.1 (K), R50.1, R51.1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: now also U7C1.6 (-); no longer U7C1.2 (-)
- net at D1.1 (K), R1.1, R2.1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: now also U3.6 (-); no longer U3.2 (-)
- net at D1.2 (A), Q2.2 (B): now also U3.7; no longer U3.1
- net at D5.1 (K), R11.1, R12.1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: now also U2.6 (-); no longer U2.2 (-)
- net at R15.1, R16.1, R17.1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: now also U6.2 (-); no longer U6.6 (-)
- net at D5.2 (A), Q1.2 (B): now also U2.7; no longer U2.1
- net at MASTER1.1, R19.1: now also U6.1; no longer U6.7
Other:
- moved on the sheet: AMP1, AMP2, AMP3, AMP4, C1, C10, C11, C12, C13, C14, C15, C16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
